File: Controller.kicad_pcb (KiCad board)
At the start: 2 copper layers, 21 x 51 mm, 36 parts, among them J1 USB_C_Receptacle_USB2.0_14P, J2 Conn_01x20, J3 Conn_01x20, J4 Conn_01x03, SW1 SW_Push, SW2 SW_Push, U1 RP2040, U2 MCP1700x-330xxTT, U3 W25Q16JVUXIQ TR, Y2 12 MHz

Commit message: Sync
Parts:
- moved SW1 32.1 mm to (90.0, 100.5), turned to 90 degrees
- moved R2 32.1 mm to (92.6, 66.0), turned to -90 degrees
- moved R7 31.2 mm to (108.5, 85.5)
- moved R1 28.7 mm to (96.0, 65.5), turned to -90 degrees
- moved C16 28.2 mm to (108.5, 78.0), turned to 180 degrees
- moved SW2 23.1 mm to (98.0, 100.5), turned to 90 degrees
- moved C8 14.1 mm to (94.0, 78.5), turned to 90 degrees
- moved R8 9.22 mm to (108.5, 82.0)
- moved C2 0.30 mm to (88.8, 87.8)
Routing:
- net GPIO0: track 0.00 -> 28.5 mm, vias 0 -> 1
- net GPIO1: track 0.00 -> 26.9 mm, vias 0 -> 1
- net GPIO2: track 0.00 -> 23.4 mm, vias 0 -> 1
- net GPIO15: track 0.00 -> 21.0 mm
- net GPIO3: track 0.00 -> 20.3 mm
- net GPIO14: track 0.00 -> 18.3 mm
- net GPIO4: track 0.00 -> 18.2 mm
- net GPIO5: track 0.00 -> 16.2 mm
- net GPIO13: track 0.00 -> 13.1 mm
- net GPIO6: track 0.00 -> 11.6 mm
- net +3V3: track 16.5 -> 27.8 mm, vias 0 -> 1
- net GPIO24: track 0.00 -> 10.3 mm
- net GPIO7: track 0.00 -> 10.2 mm
- net GPIO8: track 0.00 -> 10.2 mm, vias 0 -> 1
- net GPIO23: track 0.00 -> 8.24 mm
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